Commit message: feat: added multi-robot support - tested for upto 5 robots

File: robots/mp_400/mp_400.urdf.xacro (robot description, xacro)
@@ -99,8 +99,8 @@
     </visual>
     <collision name="body_collision">
-      <origin rpy="0 0 1.57" xyz="0.0 0.0 0.0"/>
-      <geometry>
-        <mesh filename="package://neo_simulation2/robots/mp_400/meshes/MP-400-BODY.dae" scale="0.001 0.001 0.001"/>
-        <!--cylinder length="0.381" radius="0.2545"/-->
+      <origin rpy="0 0 1.57" xyz="0.0 0.0 0.1905"/>
+      <geometry>
+        <!-- <mesh filename="package://neo_simulation2/robots/mp_400/meshes/MP-400-BODY.dae" scale="0.001 0.001 0.001"/> -->
+        <cylinder length="0.381" radius="0.2545"/>
       </geometry>
     </collision>
@@ -134,10 +134,10 @@
       </geometry>
     </visual>
-    <collision>
+    <!-- <collision>
       <origin rpy="0 0 0" xyz="0 0. 0"/>
       <geometry>
         <sphere radius="0.038"/>
       </geometry>
-    </collision>
+    </collision> -->
   </link>
   <gazebo reference="mp_400_caster_wheel_front_left_link">
@@ -170,10 +170,10 @@
       </geometry>
     </visual>
-    <collision>
+    <!-- <collision>
       <origin rpy="0 0 0" xyz="0 0. 0"/>
       <geometry>
         <sphere radius="0.038"/>
       </geometry>
-    </collision>
+    </collision> -->
   </link>
   <gazebo reference="mp_400_caster_wheel_back_left_link">
@@ -206,10 +206,10 @@
       </geometry>
     </visual>
-    <collision>
+    <!-- <collision>
       <origin rpy="0 0 0" xyz="0 0. 0"/>
       <geometry>
         <sphere radius="0.038"/>
       </geometry>
-    </collision>
+    </collision> -->
   </link>
   <gazebo reference="mp_400_caster_wheel_front_right_link">
@@ -242,10 +242,10 @@
       </geometry>
     </visual>
-    <collision>
+    <!-- <collision>
       <origin rpy="0 0 0" xyz="0 0. 0"/>
       <geometry>
         <sphere radius="0.038"/>
       </geometry>
-    </collision>
+    </collision> -->
   </link>
   <gazebo reference="mp_400_caster_wheel_back_right_link">
@@ -348,10 +348,10 @@
       </geometry>
     </visual>
-    <collision>
+    <!-- <collision>
       <origin rpy="1.57 0 0" xyz="-0.0 0 -0.06"/>
       <geometry>
         <mesh filename="package://neo_simulation2/components/sensors/SICK-MICROSCAN3.dae" scale="0.001 0.001 0.001"/>
       </geometry>
-    </collision>
+    </collision> -->
   </link>
   <!--+++++++++++++++++++ IMU ++++++++++++++++++++++++-->
